Commit message: Oppgave 3, broken

File: qube_description/urdf/qube.macro.xacro (robot description, xacro)
@@ -1,5 +1,4 @@
 <?xml version="1.0"?>
 <robot xmlns:xacro="http://www.ros.org/wiki/xacro" >
-  <xacro:property name="pi" value="3.14159265359"/>
   <!-- Definer materialer -->
   <material name="black">

Commit message: Small fixes

File: qube_description/urdf/qube.macro.xacro (robot description, xacro)
@@ -42,5 +42,5 @@
       </visual>
     </link>
-    <joint name="angle" type="revolute">
+    <joint name="motor_joint" type="revolute">
       <parent link="stator_link"/>
       <child link="rotor_link"/>

Commit message: Add parameter descriptions

File: qube_description/urdf/qube.macro.xacro (robot description, xacro)
@@ -42,10 +42,9 @@
       </visual>
     </link>
-    <joint name="motor_joint" type="revolute">
+    <joint name="motor_joint" type="continuous">
       <parent link="stator_link"/>
       <child link="rotor_link"/>
       <origin xyz="0 0 ${stator_size/2 + rotor_length/2}" rpy="0 0 0"/>
       <axis xyz="0 0 1"/>
-      <limit effort="0" velocity="0" lower="-${pi}" upper="${pi}"/>
     </joint>
     <!-- Vinkel-indikator -->

Commit message: Fix rotation in visualization

File: qube_description/urdf/qube.macro.xacro (robot description, xacro)
@@ -46,5 +46,5 @@
       <child link="rotor_link"/>
       <origin xyz="0 0 ${stator_size/2 + rotor_length/2}" rpy="0 0 0"/>
-      <axis xyz="0 0 1"/>
+      <axis xyz="0 0 -1"/>
     </joint>
     <!-- Vinkel-indikator -->
